File: Modulin.sch (KiCad schematic (older format))
At the start: 21 parts, among them J1 Conn_01x03_Male, J2 Conn_01x03_Male, J3 Conn_01x03_Female, J4 Conn_01x03_Female, U1 LM7805CT, U2 LD1117V33, U3 AD9837BCPZ-RL7, U4 MCP48FVB21-E/UN, U5 MAX4587EUB+

Commit message: Finished board Rev 1
Parts:
- U4: symbol MCP48FVB21-E/UN -> MCP48FVB21-E/UN-RESCUE-Modulin
Connections:
- net GNDA is gone; now on net GNDD: C5.2, C6.2, U3.9 (AGND)
Changed lines of the file:
@@
 EESchema Schematic File Version 2
-LIBS:74xgxx
-LIBS:74xx
+LIBS:Modulin-rescue
 LIBS:ac-dc
-LIBS:actel
 LIBS:adc-dac
-LIBS:allegro
 LIBS:Altera
 LIBS:analog_devices
@@
 LIBS:atmel
 LIBS:audio
-LIBS:battery_management
+LIBS:Battery_Management
 LIBS:bbd
 LIBS:bosch
 LIBS:brooktre
-LIBS:cmos_ieee
-LIBS:cmos4000
-LIBS:conn
+LIBS:Connector
 LIBS:contrib
 LIBS:cypress
@@
 LIBS:device
 LIBS:digital-audio
-LIBS:diode
-LIBS:display
+LIBS:Diode
+LIBS:Display
+LIBS:driver_gate
 LIBS:dsp
+LIBS:DSP_Microchip_DSPIC33
 LIBS:elec-unifil
 LIBS:ESD_Protection
+LIBS:Espressif
+LIBS:FPGA_Actel
 LIBS:ftdi
 LIBS:gennum
-LIBS:graphic_symbols
+LIBS:Graphic
 LIBS:hc11
 LIBS:infineon
@@
 LIBS:ir
 LIBS:Lattice
-LIBS:leds
+LIBS:LED
 LIBS:LEM
 LIBS:linear
+LIBS:Logic_74xgxx
+LIBS:Logic_74xx
+LIBS:Logic_CMOS_4000
+LIBS:Logic_CMOS_IEEE
 LIBS:logic_programmable
+LIBS:Logic_TTL_IEEE
 LIBS:maxim
-LIBS:mechanical
+LIBS:MCU_Microchip_PIC10
+LIBS:MCU_Microchip_PIC12
+LIBS:MCU_Microchip_PIC16
+LIBS:MCU_Microchip_PIC18
+LIBS:MCU_Microchip_PIC24
+LIBS:MCU_Microchip_PIC32
+LIBS:MCU_NXP_Kinetis
+LIBS:MCU_NXP_LPC
+LIBS:MCU_NXP_S08
+LIBS:MCU_ST_STM8
+LIBS:MCU_ST_STM32
+LIBS:MCU_Texas_MSP430
+LIBS:Mechanical
 LIBS:memory
 LIBS:microchip
-LIBS:microchip_dspic33dsc
-LIBS:microchip_pic10mcu
-LIBS:microchip_pic12mcu
-LIBS:microchip_pic16mcu
-LIBS:microchip_pic18mcu
-LIBS:microchip_pic24mcu
-LIBS:microchip_pic32mcu
 LIBS:microcontrollers
 LIBS:modules
+LIBS:Motor
 LIBS:motor_drivers
 LIBS:motorola
-LIBS:motors
-LIBS:msp430
 LIBS:nordicsemi
 LIBS:nxp
-LIBS:nxp_armmcu
 LIBS:onsemi
 LIBS:opto
@@
 LIBS:references
 LIBS:regul
-LIBS:relays
+LIBS:Relay
 LIBS:rfcom
 LIBS:RFSolutions
+LIBS:Sensor_Current
 LIBS:sensors
 LIBS:silabs
 LIBS:siliconi
-LIBS:stm8
-LIBS:stm32
 LIBS:supertex
-LIBS:switches
+LIBS:Switch
 LIBS:texas
-LIBS:transf
-LIBS:transistors
+LIBS:Transformer
+LIBS:Transistor
 LIBS:triac_thyristor
-LIBS:ttl_ieee
-LIBS:valves
+LIBS:Valve
 LIBS:video
 LIBS:wiznet
@@
 LIBS:zetex
 LIBS:Zilog
+LIBS:74xgxx
+LIBS:74xx
+LIBS:actel
+LIBS:cmos_ieee
+LIBS:cmos4000
+LIBS:conn
+LIBS:microchip_dspic33dsc
+LIBS:microchip_pic10mcu
+LIBS:microchip_pic12mcu
+LIBS:microchip_pic16mcu
+LIBS:microchip_pic18mcu
+LIBS:microchip_pic32mcu
+LIBS:msp430
+LIBS:nxp_armmcu
+LIBS:relays
+LIBS:stm8
+LIBS:stm32
+LIBS:switches
+LIBS:transf
+LIBS:transistors
+LIBS:ttl_ieee
+LIBS:valves
 LIBS:MyLib
 LIBS:Modulin-cache
@@
 $EndComp
 $Comp
-L MCP48FVB21-E/UN U4
+L MCP48FVB21-E/UN-RESCUE-Modulin U4
 U 1 1 5A0CCB1F
 P 6800 3550
@@
 F 3 "" H 4450 5550 50  0001 C CNN
 	1    4450 5550
-	-1   0    0    -1
-$EndComp
-$Comp
-L GNDA #PWR05
-U 1 1 5A0E2D61
-P 5700 5150
-F 0 "#PWR05" H 5700 4900 50  0001 C CNN
-F 1 "GNDA" H 5700 5000 50  0000 C CNN
-F 2 "" H 5700 5150 50  0001 C CNN
-F 3 "" H 5700 5150 50  0001 C CNN
-	1    5700 5150
-	-1   0    0    -1
-$EndComp
-$Comp
-L GNDA #PWR06
-U 1 1 5A0E2DAB
-P 4000 5450
-F 0 "#PWR06" H 4000 5200 50  0001 C CNN
-F 1 "GNDA" H 4000 5300 50  0000 C CNN
-F 2 "" H 4000 5450 50  0001 C CNN
-F 3 "" H 4000 5450 50  0001 C CNN
-	1    4000 5450
 	-1   0    0    -1
 $EndComp
@@
 Connection ~ 3400 700
 $Comp
-L GNDA #PWR023
-U 1 1 5A184A3D
-P 4050 900
-F 0 "#PWR023" H 4050 650 50  0001 C CNN
-F 1 "GNDA" H 4050 750 50  0000 C CNN
-F 2 "" H 4050 900 50  0001 C CNN
-F 3 "" H 4050 900 50  0001 C CNN
-	1    4050 900
-	1    0    0    -1
-$EndComp
-$Comp
-L PWR_FLAG #FLG024
-U 1 1 5A184B9B
-P 4050 900
-F 0 "#FLG024" H 4050 975 50  0001 C CNN
-F 1 "PWR_FLAG" H 4050 1050 50  0000 C CNN
-F 2 "" H 4050 900 50  0001 C CNN
-F 3 "" H 4050 900 50  0001 C CNN
-	1    4050 900
-	1    0    0    -1
-$EndComp
-$Comp
 L GNDD #PWR?
 U 1 1 5A1899B3
@@
 	1    0    0    -1
 $EndComp
+$Comp
+L GNDD #PWR?
+U 1 1 5A1B222B
+P 4000 5450
+F 0 "#PWR?" H 4000 5200 50  0001 C CNN
+F 1 "GNDD" H 4000 5325 50  0000 C CNN
+F 2 "" H 4000 5450 50  0001 C CNN
+F 3 "" H 4000 5450 50  0001 C CNN
+	1    4000 5450
+	1    0    0    -1
+$EndComp
+$Comp
+L GNDD #PWR?
+U 1 1 5A1B2483
+P 5700 5150
+F 0 "#PWR?" H 5700 4900 50  0001 C CNN
+F 1 "GNDD" H 5700 5025 50  0000 C CNN
+F 2 "" H 5700 5150 50  0001 C CNN
+F 3 "" H 5700 5150 50  0001 C CNN
+	1    5700 5150
+	1    0    0    -1
+$EndComp

Commit message: Tested basic functions of SPILib
Parts:
- U1, U2: footprint TO_SOT_Packages_THT:TO-220-3_Horizontal -> TO_SOT_Packages_THT:TO-220-3_Vertical
Changed lines of the file:
@@
 EESchema Schematic File Version 2
 LIBS:Modulin-rescue
+LIBS:74xgxx
+LIBS:74xx
 LIBS:ac-dc
+LIBS:actel
 LIBS:adc-dac
+LIBS:allegro
 LIBS:Altera
 LIBS:analog_devices
@@
 LIBS:atmel
 LIBS:audio
-LIBS:Battery_Management
+LIBS:battery_management
 LIBS:bbd
 LIBS:bosch
 LIBS:brooktre
-LIBS:Connector
+LIBS:cmos_ieee
+LIBS:cmos4000
+LIBS:conn
 LIBS:contrib
 LIBS:cypress
@@
 LIBS:device
 LIBS:digital-audio
-LIBS:Diode
-LIBS:Display
-LIBS:driver_gate
+LIBS:diode
+LIBS:display
 LIBS:dsp
-LIBS:DSP_Microchip_DSPIC33
 LIBS:elec-unifil
 LIBS:ESD_Protection
-LIBS:Espressif
-LIBS:FPGA_Actel
 LIBS:ftdi
 LIBS:gennum
-LIBS:Graphic
+LIBS:graphic_symbols
 LIBS:hc11
 LIBS:infineon
@@
 LIBS:ir
 LIBS:Lattice
-LIBS:LED
+LIBS:leds
 LIBS:LEM
 LIBS:linear
-LIBS:Logic_74xgxx
-LIBS:Logic_74xx
-LIBS:Logic_CMOS_4000
-LIBS:Logic_CMOS_IEEE
 LIBS:logic_programmable
-LIBS:Logic_TTL_IEEE
 LIBS:maxim
-LIBS:MCU_Microchip_PIC10
-LIBS:MCU_Microchip_PIC12
-LIBS:MCU_Microchip_PIC16
-LIBS:MCU_Microchip_PIC18
-LIBS:MCU_Microchip_PIC24
-LIBS:MCU_Microchip_PIC32
-LIBS:MCU_NXP_Kinetis
-LIBS:MCU_NXP_LPC
-LIBS:MCU_NXP_S08
-LIBS:MCU_ST_STM8
-LIBS:MCU_ST_STM32
-LIBS:MCU_Texas_MSP430
-LIBS:Mechanical
+LIBS:mechanical
 LIBS:memory
 LIBS:microchip
+LIBS:microchip_dspic33dsc
+LIBS:microchip_pic10mcu
+LIBS:microchip_pic12mcu
+LIBS:microchip_pic16mcu
+LIBS:microchip_pic18mcu
+LIBS:microchip_pic24mcu
+LIBS:microchip_pic32mcu
 LIBS:microcontrollers
 LIBS:modules
-LIBS:Motor
 LIBS:motor_drivers
 LIBS:motorola
+LIBS:motors
+LIBS:msp430
 LIBS:nordicsemi
 LIBS:nxp
+LIBS:nxp_armmcu
 LIBS:onsemi
 LIBS:opto
@@
 LIBS:references
 LIBS:regul
-LIBS:Relay
+LIBS:relays
 LIBS:rfcom
 LIBS:RFSolutions
-LIBS:Sensor_Current
 LIBS:sensors
 LIBS:silabs
 LIBS:siliconi
+LIBS:stm8
+LIBS:stm32
 LIBS:supertex
-LIBS:Switch
+LIBS:switches
 LIBS:texas
-LIBS:Transformer
-LIBS:Transistor
+LIBS:transf
+LIBS:transistors
 LIBS:triac_thyristor
-LIBS:Valve
+LIBS:ttl_ieee
+LIBS:valves
 LIBS:video
 LIBS:wiznet
@@
 LIBS:zetex
 LIBS:Zilog
-LIBS:74xgxx
-LIBS:74xx
-LIBS:actel
-LIBS:cmos_ieee
-LIBS:cmos4000
-LIBS:conn
-LIBS:microchip_dspic33dsc
-LIBS:microchip_pic10mcu
-LIBS:microchip_pic12mcu
-LIBS:microchip_pic16mcu
-LIBS:microchip_pic18mcu
-LIBS:microchip_pic32mcu
-LIBS:msp430
-LIBS:nxp_armmcu
-LIBS:relays
-LIBS:stm8
-LIBS:stm32
-LIBS:switches
-LIBS:transf
-LIBS:transistors
-LIBS:ttl_ieee
-LIBS:valves
 LIBS:MyLib
 LIBS:Modulin-cache
@@
 F 0 "U2" H 1800 1550 50  0000 L CNN
 F 1 "LD1117V33" H 1800 1450 50  0000 L CNN
-F 2 "TO_SOT_Packages_THT:TO-220-3_Horizontal" H 2250 1000 50  0001 L CIN
+F 2 "TO_SOT_Packages_THT:TO-220-3_Vertical" H 2250 1000 50  0001 L CIN
 F 3 "" H 2100 1200 50  0001 C CNN
 	1    2100 1200
@@
 $EndComp
 $Comp
-L GNDD #PWR08
+L GNDD #PWR05
 U 1 1 5A0E4175
 P 2100 1400
-F 0 "#PWR08" H 2100 1150 50  0001 C CNN
+F 0 "#PWR05" H 2100 1150 50  0001 C CNN
 F 1 "GNDD" H 2100 1275 50  0000 C CNN
 F 2 "" H 2100 1400 50  0001 C CNN
@@
 $EndComp
 $Comp
-L GNDD #PWR09
+L GNDD #PWR06
 U 1 1 5A0E434B
 P 1000 1100
-F 0 "#PWR09" H 1000 850 50  0001 C CNN
+F 0 "#PWR06" H 1000 850 50  0001 C CNN
 F 1 "GNDD" H 1000 975 50  0000 C CNN
 F 2 "" H 1000 1100 50  0001 C CNN
@@
 $EndComp
 $Comp
-L GNDD #PWR010
+L GNDD #PWR07
 U 1 1 5A0F163E
 P 6350 3750
-F 0 "#PWR010" H 6350 3500 50  0001 C CNN
+F 0 "#PWR07" H 6350 3500 50  0001 C CNN
 F 1 "GNDD" H 6350 3625 50  0000 C CNN
 F 2 "" H 6350 3750 50  0001 C CNN
@@
 $EndComp
 $Comp
-L GNDD #PWR011
+L GNDD #PWR08
 U 1 1 5A0F2264
 P 8300 3600
-F 0 "#PWR011" H 8300 3350 50  0001 C CNN
+F 0 "#PWR08" H 8300 3350 50  0001 C CNN
 F 1 "GNDD" H 8300 3475 50  0000 C CNN
 F 2 "" H 8300 3600 50  0001 C CNN
@@
 $EndComp
 $Comp
-L GNDD #PWR012
+L GNDD #PWR09
 U 1 1 5A0F5071
 P 9200 5450
-F 0 "#PWR012" H 9200 5200 50  0001 C CNN
+F 0 "#PWR09" H 9200 5200 50  0001 C CNN
 F 1 "GNDD" H 9200 5325 50  0000 C CNN
 F 2 "" H 9200 5450 50  0001 C CNN
@@
 $EndComp
 $Comp
-L GNDD #PWR013
+L GNDD #PWR010
 U 1 1 5A0F9668
 P 7750 5050
-F 0 "#PWR013" H 7750 4800 50  0001 C CNN
+F 0 "#PWR010" H 7750 4800 50  0001 C CNN
 F 1 "GNDD" H 7750 4925 50  0000 C CNN
 F 2 "" H 7750 5050 50  0001 C CNN
@@
 $EndSheet
 $Comp
-L GNDD #PWR015
+L GNDD #PWR011
 U 1 1 5A15B875
 P 3500 4450
-F 0 "#PWR015" H 3500 4200 50  0001 C CNN
+F 0 "#PWR011" H 3500 4200 50  0001 C CNN
 F 1 "GNDD" H 3500 4325 50  0000 C CNN
 F 2 "" H 3500 4450 50  0001 C CNN
@@
 $EndComp
 $Comp
-L GNDD #PWR016
+L GNDD #PWR012
 U 1 1 5A15B9A1
 P 3500 3650
-F 0 "#PWR016" H 3500 3400 50  0001 C CNN
+F 0 "#PWR012" H 3500 3400 50  0001 C CNN
 F 1 "GNDD" H 3500 3525 50  0000 C CNN
 F 2 "" H 3500 3650 50  0001 C CNN
@@
 F 0 "U1" H 1350 2400 50  0000 L CNN
 F 1 "LM7805CT" H 1350 2300 50  0000 L CNN
-F 2 "TO_SOT_Packages_THT:TO-220-3_Horizontal" H 1800 1850 50  0001 L CIN
+F 2 "TO_SOT_Packages_THT:TO-220-3_Vertical" H 1800 1850 50  0001 L CIN
 F 3 "" H 1650 2050 50  0001 C CNN
 	1    1650 2050
@@
 $EndComp
 $Comp
-L GNDD #PWR017
+L GNDD #PWR013
 U 1 1 5A166626
 P 1650 2250
-F 0 "#PWR017" H 1650 2000 50  0001 C CNN
+F 0 "#PWR013" H 1650 2000 50  0001 C CNN
 F 1 "GNDD" H 1650 2125 50  0000 C CNN
 F 2 "" H 1650 2250 50  0001 C CNN
@@
 Connection ~ 1150 1100
 $Comp
-L +5V #PWR018
+L +5V #PWR014
 U 1 1 5A169627
 P 2150 1950
-F 0 "#PWR018" H 2150 1800 50  0001 C CNN
+F 0 "#PWR014" H 2150 1800 50  0001 C CNN
 F 1 "+5V" H 2150 2090 50  0000 C CNN
 F 2 "" H 2150 1950 50  0001 C CNN
@@
 	8750 4850 9550 4850
 $Comp
-L PWR_FLAG #FLG019
+L PWR_FLAG #FLG015
 U 1 1 5A1721AE
 P 1150 1450
-F 0 "#FLG019" H 1150 1525 50  0001 C CNN
+F 0 "#FLG015" H 1150 1525 50  0001 C CNN
 F 1 "PWR_FLAG" H 1150 1600 50  0000 C CNN
 F 2 "" H 1150 1450 50  0001 C CNN
@@
 $EndComp
 $Comp
-L PWR_FLAG #FLG020
+L PWR_FLAG #FLG016
 U 1 1 5A17321D
 P 1150 2250
-F 0 "#FLG020" H 1150 2325 50  0001 C CNN
+F 0 "#FLG016" H 1150 2325 50  0001 C CNN
 F 1 "PWR_FLAG" H 1150 2400 50  0000 C CNN
 F 2 "" H 1150 2250 50  0001 C CNN
@@
 NoConn ~ 7950 5150
 $Comp
-L PWR_FLAG #FLG021
+L PWR_FLAG #FLG017
 U 1 1 5A177D13
 P 3350 1450
-F 0 "#FLG021" H 3350 1525 50  0001 C CNN
+F 0 "#FLG017" H 3350 1525 50  0001 C CNN
 F 1 "PWR_FLAG" H 3350 1600 50  0000 C CNN
 F 2 "" H 3350 1450 50  0001 C CNN
@@
 	3400 650  3400 900
 $Comp
-L PWR_FLAG #FLG022
+L PWR_FLAG #FLG018
 U 1 1 5A17BD80
 P 3400 700
-F 0 "#FLG022" H 3400 775 50  0001 C CNN
+F 0 "#FLG018" H 3400 775 50  0001 C CNN
 F 1 "PWR_FLAG" H 3400 850 50  0000 C CNN
 F 2 "" H 3400 700 50  0001 C CNN
@@
 Connection ~ 3400 700
 $Comp
-L GNDD #PWR?
+L GNDD #PWR019
 U 1 1 5A1899B3
 P 6100 2300
-F 0 "#PWR?" H 6100 2050 50  0001 C CNN
+F 0 "#PWR019" H 6100 2050 50  0001 C CNN
 F 1 "GNDD" H 6100 2175 50  0000 C CNN
 F 2 "" H 6100 2300 50  0001 C CNN
@@
 $EndComp
 $Comp
-L GNDD #PWR?
+L GNDD #PWR020
 U 1 1 5A189B11
 P 6650 2300
-F 0 "#PWR?" H 6650 2050 50  0001 C CNN
+F 0 "#PWR020" H 6650 2050 50  0001 C CNN
 F 1 "GNDD" H 6650 2175 50  0000 C CNN
 F 2 "" H 6650 2300 50  0001 C CNN
@@
 $EndComp
 $Comp
-L GNDD #PWR?
+L GNDD #PWR021
 U 1 1 5A1B222B
 P 4000 5450
-F 0 "#PWR?" H 4000 5200 50  0001 C CNN
+F 0 "#PWR021" H 4000 5200 50  0001 C CNN
 F 1 "GNDD" H 4000 5325 50  0000 C CNN
 F 2 "" H 4000 5450 50  0001 C CNN
@@
 $EndComp
 $Comp
-L GNDD #PWR?
+L GNDD #PWR022
 U 1 1 5A1B2483
 P 5700 5150
-F 0 "#PWR?" H 5700 4900 50  0001 C CNN
+F 0 "#PWR022" H 5700 4900 50  0001 C CNN
 F 1 "GNDD" H 5700 5025 50  0000 C CNN
 F 2 "" H 5700 5150 50  0001 C CNN
